Commit message: update xarco to use properties

File: src/my_r2d2/urdf/r2d2_model.urdf.xacro (robot description, xacro)
@@ -8,4 +8,6 @@
   <xacro:property name="wheeldiam" value="0.07" />
   <xacro:property name="pi" value="3.1415" />
+  <xacro:property name="lensr" value="0.03" />
+  <xacro:property name="lenslen" value="0.01" />
   <material name="blue">
     <color rgba="0 0 0.8 1"/>
@@ -216,12 +218,12 @@
     <visual>
      <geometry>
-         <cylinder radius="0.03" length="0.01"/>
+        <cylinder radius="${lensr}" length="${lenslen}"/>
       </geometry>
       <material name="black"/>
-      <origin rpy="1.57075 0 1.57075" xyz="0 0 0"/>
-    </visual>
-    <collision>
-      <geometry>
-        <cylinder radius="0.03" length="0.01"/>
+      <origin rpy="${pi/2} 0 ${pi/2}" xyz="0 0 0"/>
+    </visual>
+    <collision>
+      <geometry>
+        <cylinder radius="${lensr}" length="${lenslen}"/>
       </geometry>
     </collision>
