Commit message: task 3

File: src/myr2d2/urdf/test.urdf.xacro (robot description, xacro)
@@ -8,6 +8,4 @@
   <xacro:property name="wheeldiam" value="0.07" />
   <xacro:property name="pi" value="3.1415" />
-  <xacro:property name="lensr" value="0.03" />
-  <xacro:property name="lenslen" value="0.01" />
   <material name="blue">
     <color rgba="0 0 0.8 1"/>
@@ -215,23 +213,3 @@
     <origin xyz="${.707*width+0.04} 0 ${.707*width}"/>
   </joint>
-  <link name="lens">
-    <visual>
-     <geometry>
-        <cylinder radius="${lensr}" length="${lenslen}"/>
-      </geometry>
-      <material name="black"/>
-      <origin rpy="${pi/2} 0 ${pi/2}" xyz="0 0 0"/>
-    </visual>
-    <collision>
-      <geometry>
-        <cylinder radius="${lensr}" length="${lenslen}"/>
-      </geometry>
-    </collision>
-    <xacro:default_inertial mass="1"/>
-  </link>
-  <joint name="tolens" type="fixed">
-    <parent link="box"/>
-    <child link="lens"/>
-    <origin xyz="0 0 0"/>
-  </joint>
 </robot>
