Commit message: Homwork 4

File: src/myr2d2/urdf/r2d2.urdf.xacro (robot description, xacro)
@@ -215,5 +215,5 @@
 		<origin xyz="${.707*width+0.04} 0 ${.707*width}"/>
 	</joint>
-	<link name="lens">
+	<link name="lense">
 		<visual>
 			<geometry>
@@ -230,7 +230,7 @@
 		<xacro:default_inertial mass="1"/>
 	</link>
-	<joint name="tolens" type="fixed">
+	<joint name="tolense" type="fixed">
 		<parent link="box"/>
-		<child link="lens"/>
+		<child link="lense"/>
 		<origin xyz="0 0 0"/>
 	</joint>
@@ -242,3 +242,10 @@
 		<origin xyz="0 0 ${wheeldiam+bodylen/2+0.1}" />
 	</joint>
+	<link name="eye">
+	</link>
+	<joint name="tolense_eye" type="fixed">
+	<parent link="lense"/>
+	<child link="eye"/>
+	<origin xyz="${pi/2} ${-pi} ${pi/2}"/>
+	</joint>
 </robot>
